File: board/OneChipTerminal.kicad_pcb (KiCad board)
At the start: 2 copper layers, 67 x 74 mm, 33 parts, among them J1 Barrel_Jack, J2 RCAJack, J3 Conn_01x01, J4 Conn_01x01, J5 Conn_01x01, J6 Conn_01x01, J7 DB9_Male, J8 Conn_01x06, P1 Mini-DIN_6pins_ver4, U1 MAX232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

Commit message: Fixed small timing bug on CS32
Parts:
- R9: value 82R -> NC
Changed lines of the file:
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@@
       (effects (font (size 1 1) (thickness 0.15)))
     )
-    (fp_text value "82R" (at 3.81 2.37) (layer "F.Fab")
+    (fp_text value "NC" (at 3.81 2.37) (layer "F.Fab")
       (effects (font (size 1 1) (thickness 0.15)))
     )
