File: board/OneChipTerminal.kicad_sch (KiCad schematic)
At the start: 33 parts, among them J1 Barrel_Jack, J2 RCAJack, J3 Conn_01x01, J4 Conn_01x01, J5 Conn_01x01, J6 Conn_01x01, J7 DB9_Male, J8 Conn_01x06, P1 Mini-DIN_6pins_ver4, U1 MAX232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

Commit message: Fixed small timing bug on CS32
Parts:
- R9: value 82R -> NC
Changed lines of the file:
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@@
     (in_bom yes) (on_board yes)
     (property "Reference" "R9" (id 0) (at 124.46 52.832 90))
-    (property "Value" "82R" (id 1) (at 124.46 50.8 90))
+    (property "Value" "NC" (id 1) (at 124.46 50.8 90))
     (property "Footprint" "Resistor_THT:R_Axial_DIN0207_L6.3mm_D2.5mm_P7.62mm_Horizontal" (id 2) (at 124.46 49.022 90)
       (effects (font (size 1.27 1.27)) hide)
@@
     )
     (path "/00000000-0000-0000-0000-00005e61bd86"
-      (reference "R9") (unit 1) (value "82R") (footprint "Resistor_THT:R_Axial_DIN0207_L6.3mm_D2.5mm_P7.62mm_Horizontal")
+      (reference "R9") (unit 1) (value "NC") (footprint "Resistor_THT:R_Axial_DIN0207_L6.3mm_D2.5mm_P7.62mm_Horizontal")
     )
     (path "/00000000-0000-0000-0000-0000632680f1"
